Commit message: added camera

File: urdf/marrtino.urdf.xacro (robot description, xacro)
@@ -40,4 +40,5 @@
     </xacro:macro>
     <xacro:include filename="marrtino/laser.urdf.xacro"/>
+    <xacro:include filename="marrtino/camera.urdf.xacro"/>
     <link name="base_footprint">
     </link>

File: urdf/marrtino/camera.urdf.xacro (robot description, xacro)
@@ -1 +1,60 @@
-#TODO
+<robot xmlns:xacro="http://www.ros.org/wiki/xacro" name="camera">
+    <xacro:property name="cam_side" value="0.025"/>
+    <xacro:property name="cam_mass" value="0.025"/>
+    <xacro:property name="cam_h_offset" value="0.04"/>
+    <link name="camera">
+        <visual>
+            <geometry>
+                <box size="${cam_side} ${cam_side} ${cam_side}"/>
+            </geometry>
+        </visual>
+        <collision>
+            <geometry>
+                <box size="${cam_side} ${cam_side} ${cam_side}"/>
+            </geometry>
+        </collision>
+        <xacro:box_inertia m="${cam_mass}" x="${cam_side}" y="${cam_side}" z="${cam_side}"/>
+    </link>
+    <joint name="base_link_to_camera" type="fixed">
+        <parent link="base_link"/>
+        <child link="camera"/>
+        <axis xyz="1 0 0"/>
+        <origin xyz="${b_length/2 - cam_side/2} ${cam_h_offset} ${b_height/2 + cam_side/2}"/>
+    </joint>
+    <gazebo reference="camera">
+        <sensor type="camera" name="camera1">
+          <update_rate>15.0</update_rate>
+          <camera name="head">
+            <horizontal_fov>1.3962634</horizontal_fov>
+            <image>
+              <width>640</width>
+              <height>480</height>
+              <format>L8</format>
+            </image>
+            <clip>
+              <near>0.02</near>
+              <far>300</far>
+            </clip>
+            <noise>
+              <type>gaussian</type>
+              <mean>0.0</mean>
+              <stddev>0.007</stddev>
+            </noise>
+          </camera>
+          <plugin name="camera_controller" filename="libgazebo_ros_camera.so">
+            <alwaysOn>true</alwaysOn>
+            <updateRate>0.0</updateRate>
+            <cameraName>virtual_camera</cameraName>
+            <imageTopicName>image_proc</imageTopicName>
+            <cameraInfoTopicName>camera_info</cameraInfoTopicName>
+            <frameName>camera</frameName>
+            <hackBaseline>0.07</hackBaseline>
+            <distortionK1>0.0</distortionK1>
+            <distortionK2>0.0</distortionK2>
+            <distortionK3>0.0</distortionK3>
+            <distortionT1>0.0</distortionT1>
+            <distortionT2>0.0</distortionT2>
+          </plugin>
+        </sensor>
+    </gazebo>
+</robot>

Commit message: added apriltag detection in sim

File: urdf/marrtino.urdf.xacro (robot description, xacro)
@@ -1,5 +1,5 @@
 <?xml version="1.0"?>
 <robot xmlns:xacro="http://www.ros.org/wiki/xacro" name="marrtino">
-    <xacro:property name="pi_half" value="1.5707"/>
+    <xacro:property name="pi" value="3.1416"/>
     <xacro:property name="b_height" value="0.16"/>
     <xacro:property name="b_width" value="0.33"/>
@@ -41,6 +41,5 @@
     <xacro:include filename="marrtino/laser.urdf.xacro"/>
     <xacro:include filename="marrtino/camera.urdf.xacro"/>
-    <link name="base_footprint">
-    </link>
+    <link name="base_footprint"/>
     <link name="base_link">
         <visual>
@@ -104,5 +103,5 @@
         <child link="left_wheel"/>
         <axis xyz="0 0 1"/>
-        <origin xyz="${b_length/2+w_length_offset} ${+b_width/2+w_width_offset+w_height/2} ${-b_height/2-w_height_offset}" rpy="${-pi_half} 0 0"/>
+        <origin xyz="${b_length/2+w_length_offset} ${+b_width/2+w_width_offset+w_height/2} ${-b_height/2-w_height_offset}" rpy="${-pi/2} 0 0"/>
     </joint>
     <joint name="base_link_to_right_wheel" type="continuous">
@@ -110,5 +109,5 @@
         <child link="right_wheel"/>
         <axis xyz="0 0 -1"/>
-        <origin xyz="${b_length/2+w_length_offset} ${-b_width/2-w_width_offset-w_height/2} ${-b_height/2-w_height_offset}" rpy="${pi_half} 0 0"/>
+        <origin xyz="${b_length/2+w_length_offset} ${-b_width/2-w_width_offset-w_height/2} ${-b_height/2-w_height_offset}" rpy="${pi/2} 0 0"/>
     </joint>
     <joint name="base_link_to_caster_wheel" type="fixed">

File: urdf/marrtino/camera.urdf.xacro (robot description, xacro)
@@ -17,11 +17,24 @@
     </link>
     <joint name="base_link_to_camera" type="fixed">
-        <parent link="base_link"/>
-        <child link="camera"/>
-        <axis xyz="1 0 0"/>
-        <origin xyz="${b_length/2 - cam_side/2} ${cam_h_offset} ${b_height/2 + cam_side/2}"/>
+      <parent link="base_link"/>
+      <child link="camera"/>
+      <axis xyz="1 0 0"/>
+      <origin xyz="${b_length/2 - cam_side/2} ${cam_h_offset} ${b_height/2 + cam_side/2}" rpy="${-pi/2} 0 ${-pi/2}"/>
     </joint>
-    <gazebo reference="camera">
+    <!-- Gazebo e ROS utilizzano due standard differenti per l'orientamento
+      di telecamere, quindi va aggiunto un altro frame per allinearle correttamente.
+      forse si potrebbe creare un file separato per la camera sul robot reale in modo
+      da ridurre il numero di frames dato che gazevo_camera non serve.
+    -->
+    <link name="gazebo_camera"/>
+    <joint name="base_link_to_gazebo_camera" type="fixed">
+      <parent link="base_link"/>
+      <child link="gazebo_camera"/>
+      <axis xyz="1 0 0"/>
+      <origin xyz="${b_length/2 - cam_side/2} ${cam_h_offset} ${b_height/2 + cam_side/2}"/>
+    </joint>
+    <gazebo reference="gazebo_camera">
         <sensor type="camera" name="camera1">
+          <pose>0 0 0 0 0 0</pose>
           <update_rate>15.0</update_rate>
           <camera name="head">
