Commit message: -

File: urdf/marrtino/camera3.urdf.xacro (robot description, xacro)
@@ -1,3 +1,4 @@
 <robot xmlns:xacro="http://www.ros.org/wiki/xacro" name="camera">
+    <!-- upside down camera -->
     <xacro:property name="cam_side" value="0.025"/>
     <xacro:property name="cam_mass" value="0.025"/>
@@ -23,5 +24,5 @@
       <child link="camera"/>
       <axis xyz="1 0 0"/>
-      <origin xyz="${b_length/2 + cam_side/2} 0 ${cam_v_offset}" rpy="${-pi/2} 0 ${-pi/2}"/>
+      <origin xyz="${b_length/2 + cam_side/2} 0 ${cam_v_offset}" rpy="${pi/2} 0 ${pi/2}"/>
     </joint>
     <!-- Gazebo e ROS utilizzano due standard differenti per l'orientamento
@@ -35,5 +36,5 @@
       <child link="gazebo_camera"/>
       <axis xyz="1 0 0"/>
-      <origin xyz="${b_length/2 + cam_side/2} 0 ${cam_v_offset}"/>
+      <origin xyz="${b_length/2 + cam_side/2} 0 ${cam_v_offset}" rpy="${pi} 0 0"/>
     </joint>
     <gazebo reference="gazebo_camera">
